File: Pikin.kicad_pcb (KiCad board)
At the start: 2 copper layers, 254 x 160 mm, 27 parts, among them SW1 SW_Push, SW2 SW_Push, SW3 SW_Push, SW4 SW_Push, SW5 SW_Push, SW6 SW_Push, U1 brook_ufb

Commit message: Done
Parts:
- added REF**: MountingHole_3.2mm_M3, MountingHole:MountingHole_3.2mm_M3, F.Cu at (206.8, 66.5)
Changed lines of the file:
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@@
       (layerselection 0x00010fc_ffffffff)
       (disableapertmacros false)
-      (usegerberextensions false)
+      (usegerberextensions true)
       (usegerberattributes true)
-      (usegerberadvancedattributes true)
-      (creategerberjobfile true)
+      (usegerberadvancedattributes false)
+      (creategerberjobfile false)
       (svguseinch false)
       (svgprecision 6)
@@
       (psa4output false)
       (plotreference true)
-      (plotvalue true)
+      (plotvalue false)
       (plotinvisibletext false)
       (sketchpadsonfab false)
-      (subtractmaskfromsilk false)
+      (subtractmaskfromsilk true)
       (outputformat 1)
       (mirror false)
-      (drillshape 1)
+      (drillshape 0)
       (scaleselection 1)
-      (outputdirectory "")
+      (outputdirectory "Gerber/")
     )
   )
@@
     (fp_line (start -1 0.625) (end -1 -0.625) (layer "F.Fab") (width 0.1))
     (fp_line (start 1 0.625) (end -1 0.625) (layer "F.Fab") (width 0.1))
-    (pad "1" smd roundrect (at -1 0 180) (size 1.2 1.4) (layers "F.Cu" "F.Paste" "F.Mask") (roundrect_rratio 0.208333)
+    (pad "1" smd roundrect (at -1 0 180) (size 1.2 1.4) (layers "F.Cu" "F.Paste" "F.Mask") (roundrect_rratio 0.2083333333)
       (net 1 "GND") (pintype "passive"))
-    (pad "2" smd roundrect (at 1 0 180) (size 1.2 1.4) (layers "F.Cu" "F.Paste" "F.Mask") (roundrect_rratio 0.208333)
+    (pad "2" smd roundrect (at 1 0 180) (size 1.2 1.4) (layers "F.Cu" "F.Paste" "F.Mask") (roundrect_rratio 0.2083333333)
       (net 14 "Net-(R1-Pad2)") (pintype "passive"))
     (model "${KICAD6_3DMODEL_DIR}/Resistor_SMD.3dshapes/R_0805_2012Metric.wrl"
@@
     (pad "" np_thru_hole circle (at 0 0) (size 3.2 3.2) (drill 3.2) (layers *.Cu *.Mask))
   )
+  (footprint "MountingHole:MountingHole_3.2mm_M3" (layer "F.Cu")
+    (at 206.8068 66.4718)
+    (descr "Mounting Hole 3.2mm, no annular, M3")
+    (tags "mounting hole 3.2mm no annular m3")
+    (attr exclude_from_pos_files exclude_from_bom)
+    (fp_text reference "REF**" (at 0 -4.2) (layer "F.SilkS")
+      (effects (font (size 1 1) (thickness 0.15)))
+    )
+    (fp_text value "MountingHole_3.2mm_M3" (at 0 4.2) (layer "F.Fab")
+      (effects (font (size 1 1) (thickness 0.15)))
+    )
+    (fp_text user "${REFERENCE}" (at 0 0) (layer "F.Fab")
+      (effects (font (size 1 1) (thickness 0.15)))
+    )
+    (fp_circle (center 0 0) (end 3.2 0) (layer "Cmts.User") (width 0.15) (fill none))
+    (fp_circle (center 0 0) (end 3.45 0) (layer "F.CrtYd") (width 0.05) (fill none))
+    (pad "" np_thru_hole circle (at 0 0) (size 3.2 3.2) (drill 3.2) (layers *.Cu *.Mask))
+  )
   (footprint "Button_Switch_THT:SW_PUSH_6mm_H8.5mm" (layer "F.Cu")
     (at 158.04 73.95)
@@
     (fp_line (start 1 -0.625) (end 1 0.625) (layer "F.Fab") (width 0.1))
     (fp_line (start -1 0.625) (end -1 -0.625) (layer "F.Fab") (width 0.1))
-    (pad "1" smd roundrect (at -1 0) (size 1.2 1.4) (layers "F.Cu" "F.Paste" "F.Mask") (roundrect_rratio 0.208333)
+    (pad "1" smd roundrect (at -1 0) (size 1.2 1.4) (layers "F.Cu" "F.Paste" "F.Mask") (roundrect_rratio 0.2083333333)
       (net 15 "Net-(R2-Pad1)") (pintype "passive"))
-    (pad "2" smd roundrect (at 1 0) (size 1.2 1.4) (layers "F.Cu" "F.Paste" "F.Mask") (roundrect_rratio 0.208333)
+    (pad "2" smd roundrect (at 1 0) (size 1.2 1.4) (layers "F.Cu" "F.Paste" "F.Mask") (roundrect_rratio 0.2083333333)
       (net 1 "GND") (pintype "passive"))
     (model "${KICAD6_3DMODEL_DIR}/Resistor_SMD.3dshapes/R_0805_2012Metric.wrl"
@@
     )
   )
-  (gr_circle (center 101.2152 108.5816) (end 113.9652 108.5816) (layer "Dwgs.User") (width 0.2) (fill none))
-  (gr_line (start 85.7149 204.8311) (end 85.7149 78.1526) (layer "Dwgs.User") (width 0.2))
-  (gr_circle (center 328.6104 212.6159) (end 330.6104 212.6159) (layer "Dwgs.User") (width 0.2) (fill none))
-  (gr_arc (start 85.7149 78.1526) (mid 90.541211 66.55381) (end 102.170901 61.80244) (layer "Dwgs.User") (width 0.2))
-  (gr_circle (center 260.9074 103.0986) (end 273.6574 103.0986) (layer "Dwgs.User") (width 0.2) (fill none))
-  (gr_circle (center 286.9074 132.7186) (end 299.6574 132.7186) (layer "Dwgs.User") (width 0.2) (fill none))
-  (gr_line (start 229.6414 61.8236) (end 323.2524 61.8236) (layer "Dwgs.User") (width 0.2))
-  (gr_circle (center 328.8814 69.7746) (end 330.8814 69.7746) (layer "Dwgs.User") (width 0.2) (fill none))
-  (gr_circle (center 231.9074 115.1586) (end 244.6574 115.1586) (layer "Dwgs.User") (width 0.2) (fill none))
-  (gr_line (start 105.3547 70.6916) (end 200.1164 70.6916) (layer "Dwgs.User") (width 0.2))
-  (gr_circle (center 315.9074 142.3906) (end 328.6574 142.3906) (layer "Dwgs.User") (width 0.2) (fill none))
-  (gr_line (start 339.7144 78.1736) (end 339.7144 204.8311) (layer "Dwgs.User") (width 0.2))
-  (gr_arc (start 323.252222 61.823485) (mid 334.886221 66.572457) (end 339.7149 78.1736) (layer "Dwgs.User") (width 0.2))
-  (gr_arc (start 339.7149 204.8311) (mid 334.925949 216.392649) (end 323.3644 221.1816) (layer "Dwgs.User") (width 0.2))
-  (gr_arc (start 102.0654 221.1816) (mid 90.503851 216.392649) (end 85.7149 204.8311) (layer "Dwgs.User") (width 0.2))
-  (gr_circle (center 318.9074 109.9406) (end 331.6574 109.9406) (layer "Dwgs.User") (width 0.2) (fill none))
-  (gr_line (start 190.1374 61.8026) (end 229.4384 61.8026) (layer "Dwgs.User") (width 0.2))
-  (gr_circle (center 289.9074 104.0186) (end 302.6574 104.0186) (layer "Dwgs.User") (width 0.2) (fill none))
-  (gr_circle (center 157.2152 123.5816) (end 169.9652 123.5816) (layer "Dwgs.User") (width 0.2) (fill none))
-  (gr_line (start 102.1709 61.8026) (end 190.1374 61.8026) (layer "Dwgs.User") (width 0.2))
-  (gr_circle (center 96.9689 71.4046) (end 98.9689 71.4046) (layer "Dwgs.User") (width 0.2) (fill none))
-  (gr_line (start 105.3547 82.9196) (end 105.3547 70.6916) (layer "Dwgs.User") (width 0.2))
-  (gr_circle (center 172.2154 177.5819) (end 187.9654 177.5819) (layer "Dwgs.User") (width 0.2) (fill none))
-  (gr_circle (center 131.2152 108.5816) (end 143.9652 108.5816) (layer "Dwgs.User") (width 0.2) (fill none))
-  (gr_circle (center 208.6944 213.1914) (end 210.6944 213.1914) (layer "Dwgs.User") (width 0.2) (fill none))
-  (gr_line (start 200.1164 82.9196) (end 105.3547 82.9196) (layer "Dwgs.User") (width 0.2))
-  (gr_circle (center 257.9074 132.7586) (end 270.6574 132.7586) (layer "Dwgs.User") (width 0.2) (fill none))
-  (gr_circle (center 94.5249 210.7149) (end 96.5249 210.7149) (layer "Dwgs.User") (width 0.2) (fill none))
-  (gr_circle (center 228.9074 143.8486) (end 241.6574 143.8486) (layer "Dwgs.User") (width 0.2) (fill none))
-  (gr_line (start 200.1164 70.6916) (end 200.1164 82.9196) (layer "Dwgs.User") (width 0.2))
-  (gr_line (start 323.3644 221.1816) (end 102.0654 221.1816) (layer "Dwgs.User") (width 0.2))
   (gr_line (start 102.341 61.203) (end 323.425 61.2026) (layer "Edge.Cuts") (width 0.1))
   (gr_line (start 339.8834 77.661) (end 339.8834 204.745) (layer "Edge.Cuts") (width 0.1))
@@
     )
   )
-  (group "" (id 05175de8-d153-402d-8a2a-25d28fc4dd42)
-    (members
-      04e31334-0175-410a-bc85-8dd6228bea69
-      0c2d6772-605d-418a-b22a-00d8451c6824
-      0f2453f7-47cf-4157-89a6-30b47eec17fd
-      1a1f6f17-3ae7-41b7-a359-8f6ef7f1edb7
-      1f3cddaf-95c0-4656-86ed-ede4af4668c1
-      20855bdc-116d-4eb2-b5ee-c8b9ebefaab0
-      21ca7680-5650-4098-80ec-539c79ae3c4a
-      2a5ba99d-a8d2-4103-8e24-a8b3aa37b1ff
-      3e8e671a-b23f-43f2-88cd-52eca1827721
-      3f5711a9-6942-47d5-a776-bcde1cb23334
-      4eb307d7-b623-4fab-a691-2d5e0e4f3e37
-      512fd277-9de7-454a-b3d9-ab06f52cae1a
-      537a62b7-ff88-435f-aaf6-1e0429e84e7c
-      63563d42-08da-4237-8a6f-7aa4d5dfee9e
-      712463d5-56fc-4a11-a88f-f6d079aeb948
-      83f4e58e-8e79-43de-bccf-a6d767a186c1
-      93526a00-8e76-4a37-80f0-ab58fed2acf1
-      9ddc6d59-ea2f-4898-9e47-d7da9340f7bd
-      a56d8c2a-492d-492f-986e-3a417d141175
-      b3b1ccd4-a657-4a3d-8691-5506574dc6a0
-      b8818d05-0697-4aa2-b947-db693640a812
-      c4c1bec5-1dcf-436d-b0f6-b11b14e3cb89
-      c840050b-0984-4d34-a907-cdee492863f2
-      ce4dfc3f-e39b-48d7-a249-50b6350a749d
-      ced04967-57c3-4406-ac10-40f52af96afb
-      d36de82d-f117-4c0f-b89f-feb1a136f753
-      d9d035e7-3f75-4e23-9588-e6e671c6883f
-      e191fb46-dc45-4e26-882d-78bb59922927
-      e81930cd-ec3d-4f39-b139-4cba4f23d7a3
-      e86f7bef-20d4-4bc1-821e-f382fdf2812c
-      fc646187-cbc3-4dab-865a-2d2229bb2d25
-    )
-  )

Commit message: Added image files for 3D board view and layout
Parts:
- added G***: LOGO, graphics:Pikin, F.Cu at (128.0, 153.9)
- added REF**: MountingHole_3.2mm_M3, MountingHole:MountingHole_3.2mm_M3, F.Cu at (338.2, 152.2)
- added REF**: MountingHole_3.2mm_M3, MountingHole:MountingHole_3.2mm_M3, F.Cu at (74.1, 152.3)
- added U2: UP5, Brook_UFB:UP5, F.Cu at (99.2, 187.4)
- USB1: footprint Type-C:HRO-TYPE-C-31-M-12 -> Type-C:HRO-TYPE-C-31-M-12-HandSoldering
- moved REF** 20.7 mm to (76.4, 70.0)
- moved REF** 17.9 mm to (76.9, 213.4)
- moved REF** 9.15 mm to (203.5, 220.8)
- moved MX6 2.23 mm to (289.9, 102.9)
- moved U1 2.17 mm to (292.3, 188.0)
- moved REF** 2.12 mm to (329.8, 71.6)
- moved USB1 2.09 mm to (225.0, 57.5)
- moved MX1 1.70 mm to (172.5, 177.0)
- moved MX5 1.40 mm to (101.3, 107.6)
- moved MX4 1.32 mm to (260.9, 102.3)
- moved MX10 1.18 mm to (286.8, 131.9)
- moved MX11 1.05 mm to (258.1, 132.1)
- moved REF** 0.95 mm to (328.1, 213.2)
- moved MX2 0.87 mm to (232.0, 114.4)
- moved MX8 0.74 mm to (315.8, 141.3)
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Connections:
- U1 pad 25: unconnected-(U1-Pad25) -> MOSI
- U1 pad 26: unconnected-(U1-Pad26) -> SDA
- U1 pad 27: unconnected-(U1-Pad27) -> SCL
- U1 pad 28: unconnected-(U1-Pad28) -> SS
- U1 pad 29: unconnected-(U1-Pad29) -> UGND
Routing:
- net SS: track 0.00 -> 263.9 mm
- net UGND: track 0.00 -> 249.1 mm
- net SCL: track 0.00 -> 231.5 mm
- net SDA: track 0.00 -> 222.8 mm
- net MOSI: track 0.00 -> 222.4 mm
- net Left: track 252.2 -> 241.0 mm
- net Up: track 140.0 -> 144.6 mm
- net Select: track 221.3 -> 223.8 mm
- net 3K: track 118.0 -> 115.6 mm
- net TouchPad: track 210.9 -> 213.3 mm
- net RSB: track 184.3 -> 186.6 mm
- net LSB: track 192.0 -> 194.4 mm
- net Right: track 175.8 -> 178.1 mm
- net 1K: track 96.8 -> 98.9 mm
- net Net-(R2-Pad1): track 79.1 -> 81.1 mm
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Other:
- board size 254 x 160 mm -> 280.4 x 168.3 mm
